Commit message: Add imu sensor in simulation

File: go2_description/xacro/gazebo.xacro (robot description, xacro)
@@ -5,4 +5,13 @@
           <parameters>$(find quadruped_control)/config/go2_controller.yaml</parameters>
         </plugin>
+        <plugin filename="libignition-gazebo-imu-system.so" name="ignition::gazebo::systems::Imu"/>
+    </gazebo>
+    <gazebo reference="imu_link">
+        <sensor name="imu_sensor" type="imu">
+            <always_on>1</always_on>
+            <update_rate>100</update_rate>
+            <visualize>true</visualize>
+            <topic>imu</topic>
+        </sensor>
     </gazebo>
     <gazebo reference="trunk">

File: go2_description/xacro/leg.xacro (robot description, xacro)
@@ -124,5 +124,5 @@
             </inertial>
         </link>
-        <joint name="${name}_foot_fixed" type="fixed">0
+        <joint name="${name}_foot_fixed" type="fixed">
             <origin rpy="0 0 0" xyz="0 0 ${-(calf_length)}"/>
             <parent link="${name}_calf"/>

Commit message: Add lidar sensor in simulation

File: go2_description/xacro/gazebo.xacro (robot description, xacro)
@@ -3,7 +3,10 @@
     <gazebo>
         <plugin filename="ign_ros2_control-system" name="ign_ros2_control::IgnitionROS2ControlPlugin">
-          <parameters>$(find quadruped_control)/config/go2_controller.yaml</parameters>
+            <parameters>$(find quadruped_control)/config/go2_controller.yaml</parameters>
         </plugin>
         <plugin filename="libignition-gazebo-imu-system.so" name="ignition::gazebo::systems::Imu"/>
+        <plugin filename="libignition-gazebo-sensors-system.so" name="ignition::gazebo::systems::Sensors">
+            <render_engine>ogre2</render_engine>
+        </plugin>
     </gazebo>
     <gazebo reference="imu_link">
@@ -15,4 +18,39 @@
         </sensor>
     </gazebo>
+    <gazebo reference="lidar_link">
+        <sensor name='gpu_lidar' type='gpu_lidar'>"
+            <topic>lidar</topic>
+            <update_rate>4</update_rate>
+            <frame_id>lidar_link</frame_id>
+            <ray>
+                <scan>
+                    <horizontal>
+                        <samples>75</samples>
+                        <resolution>1</resolution>
+                        <min_angle>-3.141592653</min_angle>
+                        <max_angle>3.141592653</max_angle>
+                    </horizontal>
+                    <vertical>
+                        <samples>72</samples>
+                        <resolution>1</resolution>
+                        <min_angle>0.0</min_angle>
+                        <max_angle>1.570796326</max_angle>
+                    </vertical>
+                </scan>
+                <range>
+                    <min>0.05</min>
+                    <max>30.0</max>
+                    <resolution>0.01</resolution>
+                </range>
+                <noise>
+                    <type>gaussian</type>
+                    <mean>0.0</mean>
+                    <stddev>0.02</stddev>
+                </noise>
+            </ray>
+            <always_on>1</always_on>
+            <visualize>true</visualize>
+        </sensor>
+    </gazebo>
     <gazebo reference="trunk">
         <mu1>0.2</mu1>
@@ -21,9 +59,9 @@
         <kd  value="1.0"/>
     </gazebo>
-    <gazebo reference="stick_link">
+    <gazebo reference="imu_link">
         <mu1>0.2</mu1>
         <mu2>0.2</mu2>
     </gazebo>
-    <gazebo reference="imu_link">
+    <gazebo reference="lidar_link">
         <mu1>0.2</mu1>
         <mu2>0.2</mu2>

File: go2_description/xacro/robot.xacro (robot description, xacro)
@@ -76,4 +76,28 @@
         </collision>
     </link>
+    <joint name="lidar_joint" type="fixed">
+        <parent link="trunk"/>
+        <child link="lidar_link"/>
+        <origin rpy="0 2.8782 0" xyz="0.28945 0 -0.046825"/>
+    </joint>
+    <link name="lidar_link">
+        <inertial>
+            <mass value="0.001"/>
+            <origin rpy="0 0 0" xyz="0 0 0"/>
+            <inertia ixx="0.0001" ixy="0" ixz="0" iyy="0.0001" iyz="0" izz="0.0001"/>
+        </inertial>
+        <visual>
+            <origin rpy="0 0 0" xyz="0 0 0"/>
+            <geometry>
+                <sphere radius="0.045"/>
+            </geometry>
+        </visual>
+        <collision>
+            <origin rpy="0 0 0" xyz="0 0 0"/>
+            <geometry>
+                <sphere radius="0.045"/>
+            </geometry>
+        </collision>
+    </link>
     <xacro:leg name="FR" mirror="-1" mirror_dae= "False" front_hind="1"  front_hind_dae="True"  />
     <xacro:leg name="FL" mirror="1"  mirror_dae="True"   front_hind="1"  front_hind_dae="True"  />

Commit message: Add RGBD Camera in simulation

File: go2_description/xacro/gazebo.xacro (robot description, xacro)
@@ -53,4 +53,24 @@
         </sensor>
     </gazebo>
+    <gazebo reference="camera_link">
+        <sensor name="rgbd_camera" type="rgbd_camera">
+            <camera>
+                <horizontal_fov>2.0944</horizontal_fov>
+                <image>
+                    <width>1280</width>
+                    <height>720</height>
+                </image>
+                <clip>
+                    <near>0.1</near>
+                    <far>100</far>
+                </clip>
+            </camera>
+            <always_on>1</always_on>
+            <update_rate>30</update_rate>
+            <visualize>true</visualize>
+            <topic>rgbd_camera</topic>
+            <enable_metrics>true</enable_metrics>
+        </sensor>
+    </gazebo>
     <gazebo reference="trunk">
         <mu1>0.2</mu1>
@@ -64,4 +84,8 @@
     </gazebo>
     <gazebo reference="lidar_link">
+        <mu1>0.2</mu1>
+        <mu2>0.2</mu2>
+    </gazebo>
+    <gazebo reference="camera_link">
         <mu1>0.2</mu1>
         <mu2>0.2</mu2>

File: go2_description/xacro/robot.xacro (robot description, xacro)
@@ -100,4 +100,35 @@
         </collision>
     </link>
+    <joint name="camera_joint" type="fixed">
+        <parent link="trunk"/>
+        <child link="camera_link"/>
+        <origin rpy="0 0 0" xyz="0.326564 -0.000238 0.043"/>
+    </joint>
+    <link name="camera_link">
+        <inertial>
+            <mass value="0.001"/>
+            <origin rpy="0 0 0" xyz="0 0 0"/>
+            <inertia ixx="0.0001" ixy="0" ixz="0" iyy="0.0001" iyz="0" izz="0.0001"/>
+        </inertial>
+        <visual>
+            <origin rpy="0 0 0" xyz="0 0 0"/>
+            <geometry>
+                <box size="0.001 0.001 0.001"/>
+            </geometry>
+        </visual>
+        <collision>
+            <origin rpy="0 0 0" xyz="0 0 0"/>
+            <geometry>
+                <box size=".001 .001 .001"/>
+            </geometry>
+        </collision>
+    </link>
+    <joint name="camera_optical_joint" type="fixed">
+        <origin xyz="0 0 0" rpy="${-pi/2} 0 ${-pi/2}"/>
+        <parent link="camera_link"/>
+        <child link="camera_optical_link"/>
+    </joint>
+    <link name="camera_optical_link">
+    </link>
     <xacro:leg name="FR" mirror="-1" mirror_dae= "False" front_hind="1"  front_hind_dae="True"  />
     <xacro:leg name="FL" mirror="1"  mirror_dae="True"   front_hind="1"  front_hind_dae="True"  />

Commit message: inprog: Create FootSensorSystem for gazebo simulation

File: go2_description/xacro/gazebo.xacro (robot description, xacro)
@@ -5,8 +5,49 @@
             <parameters>$(find quadruped_control)/config/go2_controller.yaml</parameters>
         </plugin>
+        <plugin filename="libFootSensorSystem.so" name="gz::sim::systems::FootSensorSystem"/>
         <plugin filename="libignition-gazebo-imu-system.so" name="ignition::gazebo::systems::Imu"/>
         <plugin filename="libignition-gazebo-sensors-system.so" name="ignition::gazebo::systems::Sensors">
             <render_engine>ogre2</render_engine>
         </plugin>
+    </gazebo>
+    <gazebo reference="FR_calf">
+        <sensor name="FR_foot_contact" type="contact">
+            <update_rate>100</update_rate>
+            <always_on>1</always_on>
+            <topic>fr_foot</topic>
+            <contact>
+                <collision>FR_calf_fixed_joint_lump__FR_foot_collision_1</collision>
+            </contact>
+        </sensor>
+    </gazebo>
+    <gazebo reference="FL_calf">
+        <sensor name="FL_foot_contact" type="contact">
+            <update_rate>100</update_rate>
+            <always_on>1</always_on>
+            <topic>fl_foot</topic>
+            <contact>
+                <collision>FL_calf_fixed_joint_lump__FL_foot_collision_1</collision>
+            </contact>
+        </sensor>
+    </gazebo>
+    <gazebo reference="RR_calf">
+        <sensor name="RR_foot_contact" type="contact">
+            <update_rate>100</update_rate>
+            <always_on>1</always_on>
+            <topic>rr_foot</topic>
+            <contact>
+                <collision>RR_calf_fixed_joint_lump__RR_foot_collision_1</collision>
+            </contact>
+        </sensor>
+    </gazebo>
+    <gazebo reference="RL_calf">
+        <sensor name="RL_foot_contact" type="contact">
+            <update_rate>100</update_rate>
+            <always_on>1</always_on>
+            <topic>rl_foot</topic>
+            <contact>
+                <collision>RL_calf_fixed_joint_lump__RL_foot_collision_1</collision>
+            </contact>
+        </sensor>
     </gazebo>
     <gazebo reference="imu_link">

File: go2_description/xacro/robot.xacro (robot description, xacro)
@@ -92,4 +92,5 @@
                 <sphere radius="0.045"/>
             </geometry>
+            <material name="black"/>
         </visual>
         <collision>
